File: Design_Files/Smart_Insole_2025/Smart_insoles_2025_v1/Smart_insoles_2025_v1.kicad_sch (KiCad schematic)
At the start: 10 parts, among them U1 ESP32-C3_SUPERMINI_SMD, U2 CD74HC4067M96, U3 LSM6DSO32TR

Commit message: Added battery connector footprint. Grouping componnets in PcbNew
Parts:
- U3: footprint LSM6DSO32TR:XDCR_LSM6DSO32TR -> LDM6S032TR:XDCR_LSM6DSO32TR
Changed lines of the file:
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@@
 			)
 		)
-		(property "Footprint" "LSM6DSO32TR:XDCR_LSM6DSO32TR"
+		(property "Footprint" "LDM6S032TR:XDCR_LSM6DSO32TR"
 			(at 132.08 46.99 0)
 			(effects

Commit message: PCB new moving things around
Parts:
- C1, C2, C3: value 1uF -> 0.1uF
Changed lines of the file:
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@@
 			)
 		)
-		(property "Value" "1uF"
+		(property "Value" "0.1uF"
 			(at 226.441 41.8521 0)
 			(effects
@@
 			)
 		)
-		(property "Value" "1uF"
+		(property "Value" "0.1uF"
 			(at 215.011 41.8521 0)
 			(effects
@@
 			)
 		)
-		(property "Value" "1uF"
+		(property "Value" "0.1uF"
 			(at 237.871 41.8521 0)
 			(effects
